File: Microtransat_mainboard/estop_trigger.kicad_sch (KiCad schematic)
At the start: 3 parts

Commit message: Finished silkscreen/outline changes
Parts:
- renumbered A4 to A2, D401 to D8, R401 to R9
Changed lines of the file:
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@@
 		(dnp no)
 		(fields_autoplaced yes)
-		(property "Reference" "A4"
+		(property "Reference" "A2"
 			(at 104.14 76.2 0)
 			(effects
@@
 			(project "Microtransat_mainboard"
 				(path "/89914625-be83-416e-bb0d-b792f59b4aa6/b3769bf0-7ef3-4d04-ba3e-5e8a80f01320"
-					(reference "A4")
+					(reference "A2")
 					(unit 1)
 				)
@@
 		(dnp no)
 		(fields_autoplaced yes)
-		(property "Reference" "R401"
+		(property "Reference" "R9"
 			(at 124.46 115.5699 0)
 			(effects
@@
 			(project "Microtransat_mainboard"
 				(path "/89914625-be83-416e-bb0d-b792f59b4aa6/b3769bf0-7ef3-4d04-ba3e-5e8a80f01320"
-					(reference "R401")
+					(reference "R9")
 					(unit 1)
 				)
@@
 		(dnp no)
 		(fields_autoplaced yes)
-		(property "Reference" "#PWR0402"
+		(property "Reference" "#PWR045"
 			(at 104.14 116.84 0)
 			(effects
@@
 			(project "Microtransat_mainboard"
 				(path "/89914625-be83-416e-bb0d-b792f59b4aa6/b3769bf0-7ef3-4d04-ba3e-5e8a80f01320"
-					(reference "#PWR0402")
+					(reference "#PWR045")
 					(unit 1)
 				)
@@
 		(dnp no)
 		(fields_autoplaced yes)
-		(property "Reference" "#PWR0403"
+		(property "Reference" "#PWR046"
 			(at 121.92 132.08 0)
 			(effects
@@
 			(project "Microtransat_mainboard"
 				(path "/89914625-be83-416e-bb0d-b792f59b4aa6/b3769bf0-7ef3-4d04-ba3e-5e8a80f01320"
-					(reference "#PWR0403")
+					(reference "#PWR046")
 					(unit 1)
 				)
@@
 		(dnp no)
 		(fields_autoplaced yes)
-		(property "Reference" "D401"
+		(property "Reference" "D8"
 			(at 125.73 105.7274 90)
 			(effects
@@
 			(project "Microtransat_mainboard"
 				(path "/89914625-be83-416e-bb0d-b792f59b4aa6/b3769bf0-7ef3-4d04-ba3e-5e8a80f01320"
-					(reference "D401")
+					(reference "D8")
 					(unit 1)
 				)
@@
 		(dnp no)
 		(fields_autoplaced yes)
-		(property "Reference" "#PWR0404"
+		(property "Reference" "#PWR047"
 			(at 129.54 91.44 0)
 			(effects
@@
 			(project "Microtransat_mainboard"
 				(path "/89914625-be83-416e-bb0d-b792f59b4aa6/b3769bf0-7ef3-4d04-ba3e-5e8a80f01320"
-					(reference "#PWR0404")
-					(unit 1)
-				)
+					(reference "#PWR047")
+					(unit 1)
+				)

Commit message: Some small changes to silkscreen and component numbers
Parts:
- renumbered A2 to A501, D8 to D501, R9 to R501
Changed lines of the file:
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@@
 		(dnp no)
 		(fields_autoplaced yes)
-		(property "Reference" "A2"
+		(property "Reference" "A501"
 			(at 104.14 76.2 0)
 			(effects
@@
 			(project "Microtransat_mainboard"
 				(path "/89914625-be83-416e-bb0d-b792f59b4aa6/b3769bf0-7ef3-4d04-ba3e-5e8a80f01320"
-					(reference "A2")
+					(reference "A501")
 					(unit 1)
 				)
@@
 		(dnp no)
 		(fields_autoplaced yes)
-		(property "Reference" "R9"
+		(property "Reference" "R501"
 			(at 124.46 115.5699 0)
 			(effects
@@
 			(project "Microtransat_mainboard"
 				(path "/89914625-be83-416e-bb0d-b792f59b4aa6/b3769bf0-7ef3-4d04-ba3e-5e8a80f01320"
-					(reference "R9")
+					(reference "R501")
 					(unit 1)
 				)
@@
 		(dnp no)
 		(fields_autoplaced yes)
-		(property "Reference" "#PWR045"
+		(property "Reference" "#PWR0501"
 			(at 104.14 116.84 0)
 			(effects
@@
 			(project "Microtransat_mainboard"
 				(path "/89914625-be83-416e-bb0d-b792f59b4aa6/b3769bf0-7ef3-4d04-ba3e-5e8a80f01320"
-					(reference "#PWR045")
+					(reference "#PWR0501")
 					(unit 1)
 				)
@@
 		(dnp no)
 		(fields_autoplaced yes)
-		(property "Reference" "#PWR046"
+		(property "Reference" "#PWR0502"
 			(at 121.92 132.08 0)
 			(effects
@@
 			(project "Microtransat_mainboard"
 				(path "/89914625-be83-416e-bb0d-b792f59b4aa6/b3769bf0-7ef3-4d04-ba3e-5e8a80f01320"
-					(reference "#PWR046")
+					(reference "#PWR0502")
 					(unit 1)
 				)
@@
 		(dnp no)
 		(fields_autoplaced yes)
-		(property "Reference" "D8"
+		(property "Reference" "D501"
 			(at 125.73 105.7274 90)
 			(effects
@@
 			(project "Microtransat_mainboard"
 				(path "/89914625-be83-416e-bb0d-b792f59b4aa6/b3769bf0-7ef3-4d04-ba3e-5e8a80f01320"
-					(reference "D8")
+					(reference "D501")
 					(unit 1)
 				)
@@
 		(dnp no)
 		(fields_autoplaced yes)
-		(property "Reference" "#PWR047"
+		(property "Reference" "#PWR0503"
 			(at 129.54 91.44 0)
 			(effects
@@
 			(project "Microtransat_mainboard"
 				(path "/89914625-be83-416e-bb0d-b792f59b4aa6/b3769bf0-7ef3-4d04-ba3e-5e8a80f01320"
-					(reference "#PWR047")
-					(unit 1)
-				)
+					(reference "#PWR0503")
+					(unit 1)
+				)
