File: Microtransat_mainboard/Microtransat_mainboard.kicad_sch (KiCad schematic)
At the start: 17 parts, among them J1 Conn_01x08, J10 Conn_01x04, J101 12V IN, J2 Conn_01x04, J4 Conn_01x04, J9 Conn_01x04, SW1 SW_SPDT, U1 GPS 746, U2 SD Card Module 254, U3 IMU 4754

Commit message: Added power connector for raspberry pi
Parts:
- added J5: Conn_01x02, Connector_PinSocket_2.54mm:PinSocket_1x02_P2.54mm_Vertical, symbol Connector_Generic:Conn_01x02
Connections:
- net +5V: now also J5.1 (Pin_1)
- net GND: now also J5.2 (Pin_2)
Changed lines of the file:
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@@
+	)
+	(symbol
+		(lib_id "Connector_Generic:Conn_01x02")
+		(at 80.01 72.39 0)
+		(unit 1)
+		(exclude_from_sim no)
+		(in_bom yes)
+		(on_board yes)
+		(dnp no)
+		(fields_autoplaced yes)
+		(property "Reference" "J5"
+			(at 82.55 72.3899 0)
+			(effects
+				(font
+					(size 1.27 1.27)
+				)
+				(justify left)
+			)
+		)
+		(property "Value" "Conn_01x02"
+			(at 82.55 74.9299 0)
+			(effects
+				(font
+					(size 1.27 1.27)
+				)
+				(justify left)
+			)
+		)
+		(property "Footprint" "Connector_PinSocket_2.54mm:PinSocket_1x02_P2.54mm_Vertical"
+			(at 80.01 72.39 0)
+			(effects
+				(font
+					(size 1.27 1.27)
+				)
+				(hide yes)
+			)
+		)
+		(property "Datasheet" "~"
+			(at 80.01 72.39 0)
+			(effects
+				(font
+					(size 1.27 1.27)
+				)
+				(hide yes)
+			)
+		)
+		(property "Description" "Generic connector, single row, 01x02, script generated (kicad-library-utils/schlib/autogen/connector/)"
+			(at 80.01 72.39 0)
+			(effects
+				(font
+					(size 1.27 1.27)
+				)
+				(hide yes)
+			)
+		)
+		(pin "1"
+		)
+		(pin "2"
+		)
+		(instances
+			(project ""
+				(path "/89914625-be83-416e-bb0d-b792f59b4aa6"
+					(reference "J5")
+					(unit 1)
+				)
+			)
+		)
 	)
 	(symbol
@@
 	)
 	(symbol
+		(lib_id "power:+5V")
+		(at 74.93 72.39 90)
+		(unit 1)
+		(exclude_from_sim no)
+		(in_bom yes)
+		(on_board yes)
+		(dnp no)
+		(fields_autoplaced yes)
+		(property "Reference" "#PWR02"
+			(at 78.74 72.39 0)
+			(effects
+				(font
+					(size 1.27 1.27)
+				)
+				(hide yes)
+			)
+		)
+		(property "Value" "+5V"
+			(at 71.12 72.3899 90)
+			(effects
+				(font
+					(size 1.27 1.27)
+				)
+				(justify left)
+			)
+		)
+		(property "Footprint" ""
+			(at 74.93 72.39 0)
+			(effects
+				(font
+					(size 1.27 1.27)
+				)
+				(hide yes)
+			)
+		)
+		(property "Datasheet" ""
+			(at 74.93 72.39 0)
+			(effects
+				(font
+					(size 1.27 1.27)
+				)
+				(hide yes)
+			)
+		)
+		(property "Description" "Power symbol creates a global label with name \"+5V\""
+			(at 74.93 72.39 0)
+			(effects
+				(font
+					(size 1.27 1.27)
+				)
+				(hide yes)
+			)
+		)
+		(pin "1"
+		)
+		(instances
+			(project "Microtransat_mainboard"
+				(path "/89914625-be83-416e-bb0d-b792f59b4aa6"
+					(reference "#PWR02")
+					(unit 1)
+				)
+			)
+		)
+	)
+	(symbol
 		(lib_id "746:746")
 		(at 44.45 140.97 0)
@@
 					(unit 1)
 				)
+			)
+		)
+	)
+	(symbol
+		(lib_id "power:GND")
+		(at 74.93 74.93 270)
+		(unit 1)
+		(exclude_from_sim no)
+		(in_bom yes)
+		(on_board yes)
+		(dnp no)
+		(fields_autoplaced yes)
+		(property "Reference" "#PWR018"
+			(at 68.58 74.93 0)
+			(effects
+				(font
+					(size 1.27 1.27)
+				)
+				(hide yes)
+			)
+		)
+		(property "Value" "GND"
+			(at 71.12 74.9299 90)
+			(effects
+				(font
+					(size 1.27 1.27)
+				)
+				(justify right)
+			)
+		)
+		(property "Footprint" ""
+			(at 74.93 74.93 0)
+			(effects
+				(font
+					(size 1.27 1.27)
+				)
+				(hide yes)
+			)
+		)
+		(property "Datasheet" ""
+			(at 74.93 74.93 0)
+			(effects
+				(font
+					(size 1.27 1.27)
+				)
+				(hide yes)
+			)
+		)
+		(property "Description" "Power symbol creates a global label with name \"GND\" , ground"
+			(at 74.93 74.93 0)
+			(effects
+				(font
+					(size 1.27 1.27)
+				)
+				(hide yes)
+			)
+		)
+		(pin "1"
+		)
+		(instances
+			(project "Microtransat_mainboard"
+				(path "/89914625-be83-416e-bb0d-b792f59b4aa6"
+					(reference "#PWR018")
+					(unit 1)
+				)

Commit message: Added second RC switch for mode pin, added additional relay output, changed IMU to I2C
Connections:
- net +3V3: no longer U3.JP2_2 (P0), U3.JP2_3 (P1), U3.JP2_4 (~{RST})
- net MISO: no longer U3.JP1_5 (SDA)
- net MODE: no longer J1.5 (Pin_5)
- net MOSI: no longer U3.JP2_5 (DI)
- net SCL: now also U3.JP1_4 (SCL)
- net SCLK: no longer U3.JP1_4 (SCL)
- net SDA: now also U3.JP1_5 (SDA)
- net CS0: no longer names the net of U3.JP2_6 (CS)
- net CS0: no longer A1.12 (GPIO9)
- net CS1 renamed CS
- net CS: now also A1.12 (GPIO9); no longer A1.17 (GPIO13)
- new net MODEIN: J1.5 (Pin_5)
- new net relay0: A1.17 (GPIO13)
- no-connect marks 16 -> 21
Other:
- added sheet Mode Switch (mode_switch.kicad_sch)
- sheet Relay Board Interface ports: added relay0; removed none
Changed lines of the file:
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@@
 	)
 	(no_connect
+		(at 96.52 168.91)
+	)
+	(no_connect
 		(at 62.23 130.81)
 	)
@@
 	)
 	(no_connect
-		(at 96.52 168.91)
+		(at 96.52 161.29)
 	)
 	(no_connect
@@
 	)
 	(no_connect
+		(at 66.04 173.99)
+	)
+	(no_connect
 		(at 62.23 140.97)
 	)
@@
 	)
 	(no_connect
+		(at 66.04 168.91)
+	)
+	(no_connect
+		(at 96.52 163.83)
+	)
+	(no_connect
 		(at 118.11 154.94)
 	)
@@
 		(at 71.12 93.98)
 	)
+	(no_connect
+		(at 66.04 171.45)
+	)
 	(wire
 		(pts
@@
 		)
 	)
-	(label "MODE"
+	(label "MODEIN"
 		(at 118.11 149.86 180)
 		(effects
@@
 		)
 	)
-	(label "CS0"
-		(at 66.04 171.45 180)
+	(label "CS"
+		(at 26.67 171.45 180)
 		(effects
 			(font
@@
 		)
 	)
-	(label "CS1"
-		(at 26.67 171.45 180)
+	(label "relay0"
+		(at 246.38 48.26 180)
 		(effects
 			(font
@@
 		)
 	)
+	(label "MODEIN"
+		(at 196.85 22.86 180)
+		(effects
+			(font
+				(size 1.27 1.27)
+			)
+			(justify right bottom)
+		)
+	)
 	(label "INPWM0"
 		(at 118.11 144.78 180)
@@
 		)
 	)
-	(label "MOSI"
-		(at 66.04 173.99 180)
-		(effects
-			(font
-				(size 1.27 1.27)
-			)
-			(justify right bottom)
-		)
-	)
-	(label "SCLK"
-		(at 66.04 176.53 180)
-		(effects
-			(font
-				(size 1.27 1.27)
-			)
-			(justify right bottom)
-		)
-	)
 	(label "RX0"
 		(at 26.67 143.51 180)
@@
 		)
 	)
-	(label "MISO"
+	(label "SDA"
 		(at 66.04 179.07 180)
 		(effects
@@
 		)
 	)
-	(label "CS0"
+	(label "CS"
 		(at 194.31 107.95 180)
 		(effects
@@
 		)
 	)
-	(label "CS1"
-		(at 194.31 118.11 180)
-		(effects
-			(font
-				(size 1.27 1.27)
-			)
-			(justify right bottom)
-		)
-	)
 	(label "MOSI"
 		(at 26.67 176.53 180)
@@
 		)
 	)
+	(label "SCL"
+		(at 66.04 176.53 180)
+		(effects
+			(font
+				(size 1.27 1.27)
+			)
+			(justify right bottom)
+		)
+	)
 	(label "MODE"
 		(at 194.31 105.41 180)
@@
 		)
 	)
+	(label "MODE"
+		(at 218.44 22.86 0)
+		(effects
+			(font
+				(size 1.27 1.27)
+			)
+			(justify left bottom)
+		)
+	)
 	(label "PWM2"
 		(at 168.91 72.39 0)
@@
 		)
 	)
+	(label "relay0"
+		(at 194.31 118.11 180)
+		(effects
+			(font
+				(size 1.27 1.27)
+			)
+			(justify right bottom)
+		)
+	)
 	(label "PPS"
 		(at 62.23 143.51 0)
@@
 	)
 	(symbol
-		(lib_id "power:+3V3")
-		(at 96.52 163.83 270)
-		(unit 1)
-		(exclude_from_sim no)
-		(in_bom yes)
-		(on_board yes)
-		(dnp no)
-		(fields_autoplaced yes)
-		(property "Reference" "#PWR033"
-			(at 92.71 163.83 0)
-			(effects
-				(font
-					(size 1.27 1.27)
-				)
-				(hide yes)
-			)
-		)
-		(property "Value" "+3V3"
-			(at 100.33 163.8299 90)
-			(effects
-				(font
-					(size 1.27 1.27)
-				)
-				(justify left)
-			)
-		)
-		(property "Footprint" ""
-			(at 96.52 163.83 0)
-			(effects
-				(font
-					(size 1.27 1.27)
-				)
-				(hide yes)
-			)
-		)
-		(property "Datasheet" ""
-			(at 96.52 163.83 0)
-			(effects
-				(font
-					(size 1.27 1.27)
-				)
-				(hide yes)
-			)
-		)
-		(property "Description" "Power symbol creates a global label with name \"+3V3\""
-			(at 96.52 163.83 0)
-			(effects
-				(font
-					(size 1.27 1.27)
-				)
-				(hide yes)
-			)
-		)
-		(pin "1"
-		)
-		(instances
-			(project "Microtransat_mainboard"
-				(path "/89914625-be83-416e-bb0d-b792f59b4aa6"
-					(reference "#PWR033")
-					(unit 1)
-				)
-			)
-		)
-	)
-	(symbol
 		(lib_id "power:GND")
 		(at 217.17 135.89 0)
@@
 	)
 	(symbol
-		(lib_id "power:+3V3")
-		(at 66.04 168.91 90)
-		(unit 1)
-		(exclude_from_sim no)
-		(in_bom yes)
-		(on_board yes)
-		(dnp no)
-		(fields_autoplaced yes)
-		(property "Reference" "#PWR027"
-			(at 69.85 168.91 0)
-			(effects
-				(font
-					(size 1.27 1.27)
-				)
-				(hide yes)
-			)
-		)
-		(property "Value" "+3V3"
-			(at 62.23 168.9099 90)
-			(effects
-				(font
-					(size 1.27 1.27)
-				)
-				(justify left)
-			)
-		)
-		(property "Footprint" ""
-			(at 66.04 168.91 0)
-			(effects
-				(font
-					(size 1.27 1.27)
-				)
-				(hide yes)
-			)
-		)
-		(property "Datasheet" ""
-			(at 66.04 168.91 0)
-			(effects
-				(font
-					(size 1.27 1.27)
-				)
-				(hide yes)
-			)
-		)
-		(property "Description" "Power symbol creates a global label with name \"+3V3\""
-			(at 66.04 168.91 0)
-			(effects
-				(font
-					(size 1.27 1.27)
-				)
-				(hide yes)
-			)
-		)
-		(pin "1"
-		)
-		(instances
-			(project ""
-				(path "/89914625-be83-416e-bb0d-b792f59b4aa6"
-					(reference "#PWR027")
-					(unit 1)
-				)
-			)
-		)
-	)
-	(symbol
 		(lib_id "Connector:Conn_01x02_Pin")
 		(at 44.45 93.98 0)
@@
 	)
 	(symbol
-		(lib_id "power:+3V3")
-		(at 96.52 161.29 270)
-		(unit 1)
-		(exclude_from_sim no)
-		(in_bom yes)
-		(on_board yes)
-		(dnp no)
-		(fields_autoplaced yes)
-		(property "Reference" "#PWR030"
-			(at 92.71 161.29 0)
-			(effects
-				(font
-					(size 1.27 1.27)
-				)
-				(hide yes)
-			)
-		)
-		(property "Value" "+3V3"
-			(at 100.33 161.2899 90)
-			(effects
-				(font
-					(size 1.27 1.27)
-				)
-				(justify left)
-			)
-		)
-		(property "Footprint" ""
-			(at 96.52 161.29 0)
-			(effects
-				(font
-					(size 1.27 1.27)
-				)
-				(hide yes)
-			)
-		)
-		(property "Datasheet" ""
-			(at 96.52 161.29 0)
-			(effects
-				(font
-					(size 1.27 1.27)
-				)
-				(hide yes)
-			)
-		)
-		(property "Description" "Power symbol creates a global label with name \"+3V3\""
-			(at 96.52 161.29 0)
-			(effects
-				(font
-					(size 1.27 1.27)
-				)
-				(hide yes)
-			)
-		)
-		(pin "1"
-		)
-		(instances
-			(project "Microtransat_mainboard"
-				(path "/89914625-be83-416e-bb0d-b792f59b4aa6"
-					(reference "#PWR030")
-					(unit 1)
-				)
-			)
-		)
-	)
-	(symbol
 		(lib_id "MCU_Module:RaspberryPi_Pico")
 		(at 217.17 100.33 0)
@@
 			)
 		)
+		(pin "relay0" input
+			(at 246.38 48.26 180)
+			(effects
+				(font
+					(size 1.27 1.27)
+				)
+				(justify left)
+			)
+		)
 		(instances
 			(project "Microtransat_mainboard"
@@
 				)
 			)
+		)
+	)
+	(sheet
+		(at 196.85 20.32)
+		(size 21.59 3.81)
+		(exclude_from_sim no)
+		(in_bom yes)
+		(on_board yes)
+		(dnp no)
+		(fields_autoplaced yes)
+		(stroke
+			(width 0.1524)
+			(type solid)
+		)
+		(fill
+			(color 0 0 0 0.0000)
+		)
+		(property "Sheetname" "Mode Switch"
+			(at 196.85 19.6084 0)
+			(effects
+				(font
+					(size 1.27 1.27)
+				)
+				(justify left bottom)
+			)
+		)
+		(property "Sheetfile" "mode_switch.kicad_sch"
+			(at 196.85 24.7146 0)
+			(effects
+				(font
+					(size 1.27 1.27)
+				)
+				(justify left top)
+			)
+		)
+		(pin "OUT" output
+			(at 218.44 22.86 0)
+			(effects
+				(font
+					(size 1.27 1.27)
+				)
+				(justify right)
+			)
+		)
+		(pin "RC_IN" input
+			(at 196.85 22.86 180)
+			(effects
+				(font
+					(size 1.27 1.27)
+				)
+				(justify left)
+			)
+		)
+		(instances
+			(project "Microtransat_mainboard"
+				(path "/89914625-be83-416e-bb0d-b792f59b4aa6"
+					(page "7")
+				)
+			)

Commit message: Fixed RC Receiver pin header
Parts:
- removed J1: Conn_01x08, Connector_PinHeader_2.54mm:PinHeader_1x08_P2.54mm_Vertical, symbol Connector_Generic:Conn_01x08
- added J1: Conn_01x06, Connector_PinSocket_2.54mm:PinSocket_1x06_P2.54mm_Vertical, symbol Connector_Generic:Conn_01x06
Connections:
- net +5V: now also J1.1 (Pin_1)
- net GND: now also J1.2 (Pin_2)
- net INPWM0: now also J1.3 (Pin_3)
- net INPWM1: now also J1.4 (Pin_4)
- net MODEIN: now also J1.5 (Pin_5)
- net eSTOPIN: now also J1.6 (Pin_6)
- no-connect marks 21 -> 19
Changed lines of the file:
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@@
 	)
 	(no_connect
-		(at 118.11 157.48)
-	)
-	(no_connect
 		(at 66.04 173.99)
 	)
@@
 	)
 	(no_connect
-		(at 118.11 154.94)
-	)
-	(no_connect
 		(at 26.67 138.43)
 	)
@@
 	)
 	(symbol
+		(lib_id "Connector_Generic:Conn_01x06")
+		(at 123.19 144.78 0)
+		(unit 1)
+		(exclude_from_sim no)
+		(in_bom yes)
+		(on_board yes)
+		(dnp no)
+		(fields_autoplaced yes)
+		(property "Reference" "J1"
+			(at 125.73 144.7799 0)
+			(effects
+				(font
+					(size 1.27 1.27)
+				)
+				(justify left)
+			)
+		)
+		(property "Value" "Conn_01x06"
+			(at 125.73 147.3199 0)
+			(effects
+				(font
+					(size 1.27 1.27)
+				)
+				(justify left)
+			)
+		)
+		(property "Footprint" "Connector_PinSocket_2.54mm:PinSocket_1x06_P2.54mm_Vertical"
+			(at 123.19 144.78 0)
+			(effects
+				(font
+					(size 1.27 1.27)
+				)
+				(hide yes)
+			)
+		)
+		(property "Datasheet" "~"
+			(at 123.19 144.78 0)
+			(effects
+				(font
+					(size 1.27 1.27)
+				)
+				(hide yes)
+			)
+		)
+		(property "Description" "Generic connector, single row, 01x06, script generated (kicad-library-utils/schlib/autogen/connector/)"
+			(at 123.19 144.78 0)
+			(effects
+				(font
+					(size 1.27 1.27)
+				)
+				(hide yes)
+			)
+		)
+		(pin "3"
+		)
+		(pin "2"
+		)
+		(pin "5"
+		)
+		(pin "6"
+		)
+		(pin "1"
+		)
+		(pin "4"
+		)
+		(instances
+			(project ""
+				(path "/89914625-be83-416e-bb0d-b792f59b4aa6"
+					(reference "J1")
+					(unit 1)
+				)
+			)
+		)
+	)
+	(symbol
 		(lib_id "Connector_Generic:Conn_01x04")
 		(at 154.94 173.99 0)
@@
 					(unit 1)
 				)
-			)
-		)
-	)
-	(symbol
-		(lib_id "Connector_Generic:Conn_01x08")
-		(at 123.19 147.32 0)
-		(unit 1)
-		(exclude_from_sim no)
-		(in_bom yes)
-		(on_board yes)
-		(dnp no)
-		(fields_autoplaced yes)
-		(property "Reference" "J1"
-			(at 125.73 147.3199 0)
-			(effects
-				(font
-					(size 1.27 1.27)
-				)
-				(justify left)
-			)
-		)
-		(property "Value" "Conn_01x08"
-			(at 125.73 149.8599 0)
-			(effects
-				(font
-					(size 1.27 1.27)
-				)
-				(justify left)
-			)
-		)
-		(property "Footprint" "Connector_PinHeader_2.54mm:PinHeader_1x08_P2.54mm_Vertical"
-			(at 123.19 147.32 0)
-			(effects
-				(font
-					(size 1.27 1.27)
-				)
-				(hide yes)
-			)
-		)
-		(property "Datasheet" "~"
-			(at 123.19 147.32 0)
-			(effects
-				(font
-					(size 1.27 1.27)
-				)
-				(hide yes)
-			)
-		)
-		(property "Description" "Generic connector, single row, 01x08, script generated (kicad-library-utils/schlib/autogen/connector/)"
-			(at 123.19 147.32 0)
-			(effects
-				(font
-					(size 1.27 1.27)
-				)
-				(hide yes)
-			)
-		)
-		(pin "5"
-		)
-		(pin "1"
-		)
-		(pin "2"
-		)
-		(pin "3"
-		)
-		(pin "4"
-		)
-		(pin "6"
-		)
-		(pin "7"
-		)
-		(pin "8"
-		)
-		(instances
-			(project ""
-				(path "/89914625-be83-416e-bb0d-b792f59b4aa6"
-					(reference "J1")
-					(unit 1)
-				)

Commit message: Finished silkscreen/outline changes
Parts:
- renumbered D101 to D1, D1 to D2, J101 to J1, J5 to J2, J1 to J3, J9 to J4, J10 to J5, J4 to J6, J2 to J7, U2 to U1, U1 to U2
Connections:
- net PWM0: now also A1.20 (GPIO15); no longer A1.4 (GPIO2)
- net PWM1: now also A1.4 (GPIO2); no longer A1.19 (GPIO14)
- net PWM2: now also A1.29 (GPIO22); no longer A1.20 (GPIO15)
- net PWM3: now also A1.19 (GPIO14); no longer A1.29 (GPIO22)

Commit message: Some small changes to silkscreen and component numbers
Parts:
- renumbered A1 to A101, C1 to C101, D1 to D101, D2 to D102, J1 to J101, J2 to J102, J3 to J103, J4 to J104, J5 to J105, J6 to J106, J7 to J107, R1 to R101, R2 to R102, R3 to R103, SW1 to SW101, U1 to U101, U2 to U102, U3 to U103

Commit message: Fixed changes from design review
Parts:
- added JP1: RC3 to GPIO20, Jumper:SolderJumper-2_P1.3mm_Open_RoundedPad1.0x1.5mm, symbol Jumper:SolderJumper_2_Open
- added JP2: GPIO20 to estop, Jumper:SolderJumper-2_P1.3mm_Open_RoundedPad1.0x1.5mm, symbol Jumper:SolderJumper_2_Open
- added JP3: RC3 to estop, Jumper:SolderJumper-2_P1.3mm_Open_RoundedPad1.0x1.5mm, symbol Jumper:SolderJumper_2_Open
- J102: footprint Connector_PinSocket_2.54mm:PinSocket_1x02_P2.54mm_Vertical -> Connector_JST:JST_XH_B2B-XH-A_1x02_P2.50mm_Vertical
- J103: footprint Connector_PinSocket_2.54mm:PinSocket_1x06_P2.54mm_Vertical -> Connector_JST:JST_XH_B6B-XH-A_1x06_P2.50mm_Vertical
- R103: value 1k -> 220
Connections:
- net MODEIN is gone; now on net RC2: J103.5 (Pin_5)
- net GPIO20: now also JP1.2 (B), JP2.1 (A)
- net INPWM0 renamed RC0
- net INPWM1 renamed RC1
- net MODE renamed RC2
- net eSTOPIN renamed RC3
- net RC3: now also JP1.1 (A), JP3.1 (A)
- new net Relay Board Interface/eStopTrigger: JP2.2 (B), JP3.2 (B)
Other:
- sheet Regulators renamed Regulator
- removed sheet Mode Switch
- removed sheet eStop Trigger
