File: Microtransat_mainboard/Microtransat_mainboard.kicad_pcb (KiCad board)
At the start: 2 copper layers, 110 x 101.2 mm, 53 parts, among them J1 Conn_01x06, J101 12V IN, J102 Conn_01x02, J103 Conn_01x06, J104 Conn_01x04, J105 Conn_01x04, J106 Conn_01x04, J107 Conn_01x04, J2 Conn_01x02, J301 Conn_01x03, J302 Conn_01x03, J303 Conn_01x03, J304 Conn_01x03, J401 ESTOP IN, K401 12V SRD Form C, SW101 SW_SPDT, U101 SD Card Module 254, U102 GPS 746, U103 IMU 4754

Commit message: Fixed voltage divider/high power voltage
Parts:
- R101: value 750k -> 1M
- R102: value 500k -> 124K
- R103: value 1k -> 220
Connections:
- net +12V renamed +20V
Changed lines of the file:
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@@
 	(net 25 "/blue")
 	(net 26 "/relay0")
-	(net 27 "+12V")
+	(net 27 "+20V")
 	(net 28 "/Relay Board Interface/yellowOut")
 	(net 29 "/Relay Board Interface/eStopOut")
@@
 			)
 		)
-		(property "Value" "1k"
+		(property "Value" "220"
 			(at 0 1.83 0)
 			(layer "F.Fab")
@@
 			(layers "*.Cu" "*.Mask")
 			(remove_unused_layers no)
-			(net 27 "+12V")
+			(net 27 "+20V")
 			(pinfunction "VIN")
 			(pintype "power_in")
@@
 			(layers "*.Cu" "*.Mask")
 			(remove_unused_layers no)
-			(net 27 "+12V")
+			(net 27 "+20V")
 			(pinfunction "VIN")
 			(pintype "power_in")
@@
 			)
 		)
-		(property "Value" "500k"
+		(property "Value" "124K"
 			(at 0 1.83 90)
 			(layer "F.Fab")
@@
 			)
 		)
-		(property "Value" "750k"
+		(property "Value" "1M"
 			(at 0 1.83 90)
 			(layer "F.Fab")
@@
 			(layers "F.Cu" "F.Mask" "F.Paste")
 			(roundrect_rratio 0.192308)
-			(net 27 "+12V")
+			(net 27 "+20V")
 			(pintype "passive")
 		)
@@
 			(layers "*.Cu" "*.Mask")
 			(remove_unused_layers no)
-			(net 27 "+12V")
+			(net 27 "+20V")
 			(pinfunction "A")
 			(pintype "passive")
